File: kicad/QuackOverflow.kicad_sch (KiCad schematic)
At the start: 16 parts, among them J1 Qi_Reciever, J2 USB_C_Receptacle_USB2.0_14P, U2 TP4056-42-ESOP8, U3 ESP32-C3-WROOM-02

Commit message: Revert "renamed pcb cuz i realized i needed to make another"
This reverts commit 06b52c8c19761527b94a53c6af2c4550971bfb81.
Parts:
- removed J2: USB_C_Receptacle_USB2.0_14P, Connector_USB:USB_C_Receptacle_HRO_TYPE-C-31-M-12, symbol Connector:USB_C_Receptacle_USB2.0_14P
- removed R3, R4: 5.1k, Resistor_SMD:R_1206_3216Metric_Pad1.30x1.75mm_HandSolder, symbol Device:R
- removed U3: ESP32-C3-WROOM-02, Espressif:ESP32-C3-WROOM-02, symbol Espressif:ESP32-C3-WROOM-02
- added U1: ESP32-C3-MINI-1, Espressif:ESP32-C3-MINI-1, symbol Espressif:ESP32-C3-MINI-1
Connections:
- net CHRG: now also U1.23 (GPIO9)
- net GND: now also U1.1 (GND), U1.11 (GND), U1.14 (GND), U1.2 (GND), U1.36 (GND), U1.37 (GND), U1.38 (GND), U1.39 (GND), U1.40 (GND), U1.41 (GND), U1.42 (GND), U1.43 (GND), U1.44 (GND), U1.45 (GND), U1.46 (GND), U1.47 (GND), U1.48 (GND), U1.49 (GND), U1.50 (GND), U1.51 (GND), U1.52 (GND), U1.53 (GND)
- net LEDS: now also U1.22 (GPIO8)
- net VBAT: now also U1.3 (3V3)
- net at R1.2: now also U1.8 (EN/CHIP_PU)
- net 5V_IN renamed QI_5V
