File: kicad/duck-pcb/duck_pcb.kicad_sch (KiCad schematic)
At the start: 13 parts, among them J1 Qi_Reciever, U1 ESP32-C3-MINI-1, U2 TP4056-42-ESOP8

Commit message: holy moly i almost lost everything
Parts:
- removed U1: ESP32-C3-MINI-1, Espressif:ESP32-C3-MINI-1, symbol Espressif:ESP32-C3-MINI-1
- added J2: USB_C_Receptacle_USB2.0_14P, Connector_USB:USB_C_Receptacle_HRO_TYPE-C-31-M-12, symbol Connector:USB_C_Receptacle_USB2.0_14P
- added R3, R4: 5.1k, Resistor_SMD:R_1206_3216Metric_Pad1.30x1.75mm_HandSolder, symbol Device:R
- added U3: ESP32-C3-WROOM-02, Espressif:ESP32-C3-WROOM-02, symbol Espressif:ESP32-C3-WROOM-02
Connections:
- net CHRG: now also U3.8 (GPIO9)
- net GND: now also J2.A1 (GND), J2.A12 (GND), J2.B1 (GND), J2.B12 (GND), J2.S1 (SHIELD), R3.2, R4.2, U3.19 (GND), U3.9 (GND)
- net LEDS: now also U3.7 (GPIO8)
- net VBAT: now also U3.1 (3V3)
- net at R1.2: now also U3.2 (EN/CHIP_PU)
- net QI_5V renamed 5V_IN
- net 5V_IN: now also J2.A4 (VBUS), J2.A9 (VBUS), J2.B4 (VBUS), J2.B9 (VBUS)
- new net: J2.B5 (CC2), R4.1
- new net: J2.A5 (CC1), R3.1
- new net USB_D+: J2.A6 (D+), U3.14 (GPIO19/USB_D+)
- new net USB_D-: J2.A7 (D-), U3.13 (GPIO18/USB_D-)
